File: Akashi-07.kicad_pcb (KiCad board)
At the start: 2 copper layers, 68.6 x 53.3 mm, 47 parts, among them J1 Conn_Coaxial, J2 Screw_Terminal_01x02, J3 SJ1-3533, J4 Conn_01x08, J5 Conn_01x06, J6 Conn_01x10, J7 Conn_01x08, U1 Si5351A-B-GT, U2 SN74LVC74APW, U3 TS5A23157DGSR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

Commit message: update BOM
Parts:
- L1: footprint Resistors_THT:R_Axial_DIN0204_L3.6mm_D1.6mm_P2.54mm_Vertical -> Inductors_THT:L_Axial_L7.0mm_D3.3mm_P5.08mm_Vertical_Fastron_MICC
Routing:
- net Net-(C5-Pad1): track 25.7 -> 23.2 mm
Other:
- board text added: "Akashi-07 : (C) 2020 Seiichi Horie QSD prototype ver 1.0 https://github.com/suikan4github/Akashi-07"
- board text removed: "Akashi-07 : (C) 2020 Seiichi Horie https://github.com/suikan4github/Akashi-07"
Changed lines of the file:
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@@
     (add_net VDD)
+  )
+  (module Inductors_THT:L_Axial_L7.0mm_D3.3mm_P5.08mm_Vertical_Fastron_MICC (layer F.Cu)
+    (at 164.465 93.98 270)
+    (descr "L, Axial series, Axial, Vertical, pin pitch=5.08mm, , length*diameter=7*3.3mm^2, Fastron, MICC, http://www.fastrongroup.com/image-show/70/MICC.pdf?type=Complete-DataSheet&productType=series")
+    (tags "L Axial series Axial Vertical pin pitch 5.08mm  length 7mm diameter 3.3mm Fastron MICC")
+    (fp_text reference L1 (at 2.54 -2.71 90) (layer F.SilkS)
+      (effects (font (size 1 1) (thickness 0.15)))
+    )
+    (fp_text value 10mH (at 2.54 2.71 90) (layer F.Fab)
+      (effects (font (size 1 1) (thickness 0.15)))
+    )
+    (fp_circle (center 0 0) (end 1.65 0) (layer F.Fab) (width 0.1))
+    (fp_circle (center 0 0) (end 1.71 0) (layer F.SilkS) (width 0.12))
+    (fp_line (start 0 0) (end 5.08 0) (layer F.Fab) (width 0.1))
+    (fp_line (start 1.71 0) (end 3.98 0) (layer F.SilkS) (width 0.12))
+    (fp_line (start -2 -2) (end -2 2) (layer F.CrtYd) (width 0.05))
+    (fp_line (start -2 2) (end 6.2 2) (layer F.CrtYd) (width 0.05))
+    (fp_line (start 6.2 2) (end 6.2 -2) (layer F.CrtYd) (width 0.05))
+    (fp_line (start 6.2 -2) (end -2 -2) (layer F.CrtYd) (width 0.05))
+    (pad 1 thru_hole circle (at 0 0 270) (size 1.6 1.6) (drill 0.8) (layers *.Cu *.Mask)
+      (net 7 "Net-(C6-Pad1)"))
+    (pad 2 thru_hole oval (at 5.08 0 270) (size 1.6 1.6) (drill 0.8) (layers *.Cu *.Mask)
+      (net 5 "Net-(C5-Pad1)"))
+    (model Inductors_THT.3dshapes/L_Axial_L7.0mm_D3.3mm_P5.08mm_Vertical_Fastron_MICC.wrl
+      (at (xyz 0 0 0))
+      (scale (xyz 0.393701 0.393701 0.393701))
+      (rotate (xyz 0 0 0))
+    )
   )
   (module TO_SOT_Packages_SMD:SOT-89-3_Handsoldering (layer F.Cu)
@@
     (pad 2 thru_hole oval (at 2.54 0 180) (size 1.4 1.4) (drill 0.7) (layers *.Cu *.Mask)
       (net 13 /connector/SDA))
-    (model ${KISYS3DMOD}/Resistors_THT.3dshapes/R_Axial_DIN0204_L3.6mm_D1.6mm_P2.54mm_Vertical.wrl
-      (at (xyz 0 0 0))
-      (scale (xyz 0.393701 0.393701 0.393701))
-      (rotate (xyz 0 0 0))
-    )
-  )
-  (module Resistors_THT:R_Axial_DIN0204_L3.6mm_D1.6mm_P2.54mm_Vertical (layer F.Cu)
-    (at 164.465 93.98 270)
-    (descr "Resistor, Axial_DIN0204 series, Axial, Vertical, pin pitch=2.54mm, 0.16666666666666666W = 1/6W, length*diameter=3.6*1.6mm^2, http://cdn-reichelt.de/documents/datenblatt/B400/1_4W%23YAG.pdf")
-    (tags "Resistor Axial_DIN0204 series Axial Vertical pin pitch 2.54mm 0.16666666666666666W = 1/6W length 3.6mm diameter 1.6mm")
-    (fp_text reference L1 (at 1.27 -1.86 90) (layer F.SilkS)
-      (effects (font (size 1 1) (thickness 0.15)))
-    )
-    (fp_text value 10mH (at 1.27 1.86 90) (layer F.Fab)
-      (effects (font (size 1 1) (thickness 0.15)))
-    )
-    (fp_circle (center 0 0) (end 0.8 0) (layer F.Fab) (width 0.1))
-    (fp_circle (center 0 0) (end 0.86 0) (layer F.SilkS) (width 0.12))
-    (fp_line (start 0 0) (end 2.54 0) (layer F.Fab) (width 0.1))
-    (fp_line (start 0.86 0) (end 1.54 0) (layer F.SilkS) (width 0.12))
-    (fp_line (start -1.15 -1.15) (end -1.15 1.15) (layer F.CrtYd) (width 0.05))
-    (fp_line (start -1.15 1.15) (end 3.55 1.15) (layer F.CrtYd) (width 0.05))
-    (fp_line (start 3.55 1.15) (end 3.55 -1.15) (layer F.CrtYd) (width 0.05))
-    (fp_line (start 3.55 -1.15) (end -1.15 -1.15) (layer F.CrtYd) (width 0.05))
-    (pad 1 thru_hole circle (at 0 0 270) (size 1.4 1.4) (drill 0.7) (layers *.Cu *.Mask)
-      (net 7 "Net-(C6-Pad1)"))
-    (pad 2 thru_hole oval (at 2.54 0 270) (size 1.4 1.4) (drill 0.7) (layers *.Cu *.Mask)
-      (net 5 "Net-(C5-Pad1)"))
     (model ${KISYS3DMOD}/Resistors_THT.3dshapes/R_Axial_DIN0204_L3.6mm_D1.6mm_P2.54mm_Vertical.wrl
       (at (xyz 0 0 0))
@@
     (effects (font (size 1 1) (thickness 0.15)))
   )
-  (gr_text Akashi-07 (at 128.27 123.19) (layer F.SilkS)
+  (gr_text Akashi-07 (at 144.78 80.01) (layer F.SilkS)
     (effects (font (size 1.5 1.5) (thickness 0.2)))
   )
-  (gr_text "Akashi-07 : (C) 2020 Seiichi Horie\nhttps://github.com/suikan4github/Akashi-07\n" (at 144.145 81.28) (layer B.SilkS)
+  (gr_text "Akashi-07 : (C) 2020 Seiichi Horie\nQSD prototype ver 1.0\nhttps://github.com/suikan4github/Akashi-07\n" (at 143.51 81.28) (layer B.SilkS)
     (effects (font (size 1 1) (thickness 0.15)) (justify mirror))
   )
@@
   (segment (start 127.08 88.9) (end 120.77 82.59) (width 0.25) (layer F.Cu) (net 4))
   (segment (start 167.005 102.87) (end 164.465 100.33) (width 0.25) (layer F.Cu) (net 5))
-  (segment (start 164.465 100.33) (end 164.465 96.52) (width 0.25) (layer F.Cu) (net 5))
   (segment (start 149.2247 100) (end 150.2139 100) (width 0.25) (layer F.Cu) (net 5))
   (segment (start 150.2139 100) (end 150.2139 101) (width 0.25) (layer F.Cu) (net 5))
@@
   (segment (start 164.465 100.33) (end 162.834 101.961) (width 0.25) (layer F.Cu) (net 5))
   (segment (start 150.2139 101) (end 149.2247 101) (width 0.25) (layer F.Cu) (net 5))
+  (segment (start 164.465 100.33) (end 164.465 99.06) (width 0.25) (layer F.Cu) (net 5))
   (segment (start 175.26 106.125) (end 172.005 102.87) (width 0.25) (layer B.Cu) (net 6))
   (segment (start 175.26 109.22) (end 175.26 106.125) (width 0.25) (layer B.Cu) (net 6))

Commit message: Ready for FusionPCB and Digikey
Connections:
- X1 pad 1: Net-(X1-Pad1) -> VDD
Changed lines of the file:
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@@
   (general
     (thickness 1.6)
-    (drawings 17)
+    (drawings 18)
     (tracks 270)
     (zones 0)
     (modules 47)
-    (nets 54)
+    (nets 53)
   )
   (page A4)
@@
     (visible_elements FFFFFF7F)
     (pcbplotparams
-      (layerselection 0x010fc_ffffffff)
-      (usegerberextensions false)
+      (layerselection 0x010f0_ffffffff)
+      (usegerberextensions true)
       (usegerberattributes true)
       (usegerberadvancedattributes true)
-      (creategerberjobfile true)
+      (creategerberjobfile false)
       (excludeedgelayer true)
       (linewidth 0.100000)
@@
       (outputformat 1)
       (mirror false)
-      (drillshape 1)
+      (drillshape 0)
       (scaleselection 1)
       (outputdirectory ""))
@@
   (net 51 "Net-(U1-Pad3)")
   (net 52 "Net-(U2-Pad6)")
-  (net 53 "Net-(X1-Pad1)")
   (net_class Default "This is the default net class."
     (clearance 0.2)
@@
     (add_net "Net-(U2-Pad2)")
     (add_net "Net-(U2-Pad6)")
-    (add_net "Net-(X1-Pad1)")
     (add_net VDD)
   )
@@
     )
     (pad 1 smd rect (at -2.63 2.6 270) (size 1.98 3) (layers F.Cu F.Paste F.Mask)
-      (net 53 "Net-(X1-Pad1)"))
+      (net 1 VDD))
     (pad 2 smd rect (at 2.63 2.6 270) (size 1.98 3) (layers F.Cu F.Paste F.Mask)
       (net 2 GND))
@@
     )
   )
+  (dimension 4.064 (width 0.15) (layer Dwgs.User)
+    (gr_text "160 mils" (at 155.448 69.312) (layer Dwgs.User)
+      (effects (font (size 1 1) (thickness 0.15)))
+    )
+    (feature1 (pts (xy 153.416 73.66) (xy 153.416 70.025579)))
+    (feature2 (pts (xy 157.48 73.66) (xy 157.48 70.025579)))
+    (crossbar (pts (xy 157.48 70.612) (xy 153.416 70.612)))
+    (arrow1a (pts (xy 153.416 70.612) (xy 154.542504 70.025579)))
+    (arrow1b (pts (xy 153.416 70.612) (xy 154.542504 71.198421)))
+    (arrow2a (pts (xy 157.48 70.612) (xy 156.353496 70.025579)))
+    (arrow2b (pts (xy 157.48 70.612) (xy 156.353496 71.198421)))
+  )
   (gr_text "JP1,2\n1-2 : Ref\n2-3 : Sig" (at 127 118.11) (layer F.SilkS)
