File: Akashi-07.kicad_pcb (KiCad board)
At the start: 2 copper layers, 68.6 x 53.3 mm, 47 parts, among them J1 Conn_Coaxial, J2 Screw_Terminal_01x02, J3 SJ1-3533, J4 Conn_01x08, J5 Conn_01x06, J6 Conn_01x10, J7 Conn_01x08, U1 Si5351A-B-GT, U2 SN74LVC74APW, U3 TS5A23157DGSR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

Commit message: Update readme
Parts:
- U5: value TA48L033 -> TLV73333PDBV; footprint TO_SOT_Packages_SMD:SOT-89-3_Handsoldering -> TO_SOT_Packages_SMD:SOT-23-5_HandSoldering
- moved U5 1.93 mm to (157.5, 116.2), turned to 0 degrees
Connections:
- U5 pad 1: VDD -> Net-(C16-Pad1)
Routing:
- net VDD: track 85.4 -> 93.9 mm
- net GND: track 17.2 -> 9.01 mm, vias 7 -> 8
- net Net-(C16-Pad1): track 21.4 -> 28.1 mm
Other:
- board text added: "1"
- board text added: "Akashi-07 : (C) 2020 Seiichi Horie QSD prototype ver 1.0.1 https://github.com/suikan4github/Akashi-07"
- board text removed: "Akashi-07 : (C) 2020 Seiichi Horie QSD prototype ver 1.0 https://github.com/suikan4github/Akashi-07"
