File: signal.sch (KiCad schematic (older format))
At the start: 38 parts, among them J1 Conn_Coaxial, J2 Screw_Terminal_01x02, J3 SJ1-3533, U1 Si5351A-B-GT, U2 SN74LVC74APW, U3 TS5A23157DGSR, U4 AD8032ANZ, X1 CSX-750FBC25000000T

Commit message: BOM is ready
Parts:
- J2: DigiKey (none) -> 281-2888-ND
- J3: DigiKey (none) -> CP1-3533N-ND
- L1: DigiKey (none) -> 495-5590-1-ND
- U1: DigiKey (none) -> 336-2399-5-ND
- U2: DigiKey (none) -> 296-1241-1-ND
- U3: DigiKey (none) -> 296-17076-1-ND
- U4: DigiKey (none) -> AD8032ANZ-ND
- X1: DigiKey (none) -> 300-7246-1-ND
Changed lines of the file:
@@
 F 2 "Housings_SSOP:MSOP-10_3x3mm_Pitch0.5mm" H 3000 3950 50  0001 C CNN
 F 3 "https://www.silabs.com/documents/public/data-sheets/Si5351-B.pdf" H 2650 4650 50  0001 C CNN
+F 4 "336-2399-5-ND" H 3000 4750 50  0001 C CNN "DigiKey"
 	1    3000 4750
 	1    0    0    -1
@@
 F 2 "Oscillators:Oscillator_SMD_SeikoEpson_SG8002CA-4pin_7.0x5.0mm_HandSoldering" H 2300 4100 50  0001 C CNN
 F 3 "https://www.digikey.jp/product-detail/ja/citizen-finedevice-co-ltd/CSX-750FBC25000000T/300-7246-1-ND/482134" H 1500 4450 50  0001 C CNN
+F 4 "300-7246-1-ND" H 1600 4450 50  0001 C CNN "DigiKey"
 	1    1600 4450
 	1    0    0    -1
@@
 F 2 "Housings_SSOP:TSSOP-14_4.4x5mm_Pitch0.65mm" H 4700 4550 50  0001 C CNN
 F 3 "https://www.tij.co.jp/product/jp/SN74LVC74A" H 4700 4550 50  0001 C CNN
+F 4 "296-1241-1-ND" H 4700 4550 50  0001 C CNN "DigiKey"
 	1    4700 4550
 	1    0    0    -1
@@
 F 2 "Housings_SSOP:TSSOP-14_4.4x5mm_Pitch0.65mm" H 6850 5350 50  0001 C CNN
 F 3 "https://www.tij.co.jp/product/jp/SN74LVC74A" H 6850 5350 50  0001 C CNN
+F 4 "296-1241-1-ND" H 6850 5350 50  0001 C CNN "DigiKey"
 	3    6850 5350
 	1    0    0    -1
@@
 F 2 "Housings_DIP:DIP-8_W7.62mm" H 9500 2700 50  0001 C CNN
 F 3 "https://www.analog.com/media/en/technical-documentation/data-sheets/AD8031_8032.pdf" H 9650 2850 50  0001 C CNN
+F 4 "AD8032ANZ-ND" H 9400 2700 50  0001 C CNN "DigiKey"
 	1    9400 2700
 	1    0    0    -1
@@
 F 2 "Housings_DIP:DIP-8_W7.62mm" H 9500 3700 50  0001 C CNN
 F 3 "https://www.analog.com/media/en/technical-documentation/data-sheets/AD8031_8032.pdf" H 9650 3850 50  0001 C CNN
+F 4 "AD8032ANZ-ND" H 9400 3700 50  0001 C CNN "DigiKey"
 	2    9400 3700
 	1    0    0    -1
@@
 F 2 "Housings_DIP:DIP-8_W7.62mm" H 9200 5300 50  0001 C CNN
 F 3 "https://www.analog.com/media/en/technical-documentation/data-sheets/AD8031_8032.pdf" H 9350 5450 50  0001 C CNN
+F 4 "AD8032ANZ-ND" H 9100 5300 50  0001 C CNN "DigiKey"
 	3    9100 5300
 	1    0    0    -1
@@
 F 2 "Resistors_THT:R_Axial_DIN0204_L3.6mm_D1.6mm_P2.54mm_Vertical" H 4450 1850 50  0001 C CNN
 F 3 "https://www.digikey.jp/product-detail/en/tdk-electronics-inc/B82144A2106J000/495-5615-1-ND/4245955" H 4450 1850 50  0001 C CNN
+F 4 "495-5590-1-ND" H 4450 1850 50  0001 C CNN "DigiKey"
 	1    4450 1850
 	1    0    0    -1
@@
 F 2 "Connectors_Terminal_Blocks:TerminalBlock_bornier-2_P5.08mm" H 2950 2750 50  0001 C CNN
 F 3 "~" H 2950 2750 50  0001 C CNN
+F 4 "281-2888-ND" H 2950 2750 50  0001 C CNN "DigiKey"
 	1    2950 2750
 	-1   0    0    -1
@@
 F 2 "Housings_SSOP:TSSOP-14_4.4x5mm_Pitch0.65mm" H 4700 5600 50  0001 C CNN
 F 3 "https://www.tij.co.jp/product/jp/SN74LVC74A" H 4700 5600 50  0001 C CNN
+F 4 "296-1241-1-ND" H 4700 5600 50  0001 C CNN "DigiKey"
 	2    4700 5600
 	1    0    0    -1
@@
 F 2 "project_lib:Jack_3.5mm_CUI_SJ1-3533NG_Horizontal_CircularHoles" H 10650 3250 50  0001 C CNN
 F 3 "https://www.digikey.jp/product-detail/ja/cui-devices/SJ1-3533/CP1-3533-ND/738695" H 10650 3250 50  0001 C CNN
+F 4 "CP1-3533N-ND" H 10650 3250 50  0001 C CNN "DigiKey"
 	1    10650 3250
 	-1   0    0    -1
@@
 F 2 "project_lib:TS5A23157DGSR" H 6650 2840 60  0001 C CNN
 F 3 "https://www.tij.co.jp/product/jp/TS5A23157" H 5850 2500 60  0001 C CNN
+F 4 "296-17076-1-ND" H 5850 2500 50  0001 C CNN "DigiKey"
 	1    5850 2500
 	1    0    0    -1

Commit message: update BOM
Parts:
- J1: DigiKey (none) -> WM5543-ND
- L1: footprint Resistors_THT:R_Axial_DIN0204_L3.6mm_D1.6mm_P2.54mm_Vertical -> Inductors_THT:L_Axial_L7.0mm_D3.3mm_P5.08mm_Vertical_Fastron_MICC; DigiKey 495-5590-1-ND -> AIAP-01-102K-TCT-ND
Other:
- note added: "Abracon AIAP-01-102K-T\nAIAP-01-102K-TCT-ND \n\n"
- note removed: "B82144A2106J000"
Changed lines of the file:
@@
 F 0 "L1" H 4503 1896 50  0000 L CNN
 F 1 "10mH" H 4503 1805 50  0000 L CNN
-F 2 "Resistors_THT:R_Axial_DIN0204_L3.6mm_D1.6mm_P2.54mm_Vertical" H 4450 1850 50  0001 C CNN
+F 2 "Inductors_THT:L_Axial_L7.0mm_D3.3mm_P5.08mm_Vertical_Fastron_MICC" H 4450 1850 50  0001 C CNN
 F 3 "https://www.digikey.jp/product-detail/en/tdk-electronics-inc/B82144A2106J000/495-5615-1-ND/4245955" H 4450 1850 50  0001 C CNN
-F 4 "495-5590-1-ND" H 4450 1850 50  0001 C CNN "DigiKey"
+F 4 "AIAP-01-102K-TCT-ND" H 4450 1850 50  0001 C CNN "DigiKey"
 	1    4450 1850
 	1    0    0    -1
@@
 F 2 "Connectors:SMA_THT_Jack_Straight" H 2950 1750 50  0001 C CNN
 F 3 " ~" H 2950 1750 50  0001 C CNN
+F 4 "WM5543-ND" H 2950 1750 50  0001 C CNN "DigiKey"
 	1    2950 1750
 	-1   0    0    -1
@@
 Wire Wire Line
 	5400 5500 5400 3200
-Text Notes 3950 1600 0    50   ~ 0
-B82144A2106J000
+Text Notes 3800 1950 0    50   ~ 0
+Abracon AIAP-01-102K-T\nAIAP-01-102K-TCT-ND	\n\n
 $Comp
 L Connector:TestPoint TP1

Commit message: Ready for FusionPCB and Digikey
Connections:
- net VDD: now also X1.1 (OE)
- no-connect marks 3 -> 2
Other:
- moved on the sheet: C1
Changed lines of the file:
@@
 L Device:C C1
 U 1 1 5F0E05E9
-P 1400 3750
-F 0 "C1" H 1150 3800 50  0000 L CNN
-F 1 "0.1u" H 1100 3700 50  0000 L CNN
-F 2 "Capacitors_THT:C_Disc_D4.7mm_W2.5mm_P5.00mm" H 1438 3600 50  0001 C CNN
-F 3 "~" H 1400 3750 50  0001 C CNN
-	1    1400 3750
-	1    0    0    -1
-$EndComp
-Wire Wire Line
-	1600 4150 1600 3550
-Wire Wire Line
-	1400 3600 1400 3550
-Wire Wire Line
-	1400 3550 1600 3550
+P 1750 3800
+F 0 "C1" H 1450 3850 50  0000 L CNN
+F 1 "0.1u" H 1400 3750 50  0000 L CNN
+F 2 "Capacitors_THT:C_Disc_D4.7mm_W2.5mm_P5.00mm" H 1788 3650 50  0001 C CNN
+F 3 "~" H 1750 3800 50  0001 C CNN
+	1    1750 3800
+	1    0    0    -1
+$EndComp
+Wire Wire Line
+	1600 4150 1600 4000
+Wire Wire Line
+	1750 3650 1750 3550
+Wire Wire Line
+	1750 3550 1600 3550
 Connection ~ 1600 3550
 Wire Wire Line
@@
 L power:GND #PWR01
 U 1 1 5F0E05F4
-P 1400 4000
-F 0 "#PWR01" H 1400 3750 50  0001 C CNN
-F 1 "GND" H 1405 3827 50  0000 C CNN
-F 2 "" H 1400 4000 50  0001 C CNN
-F 3 "" H 1400 4000 50  0001 C CNN
-	1    1400 4000
-	1    0    0    -1
-$EndComp
-Wire Wire Line
-	1400 3900 1400 4000
+P 1750 4000
+F 0 "#PWR01" H 1750 3750 50  0001 C CNN
+F 1 "GND" H 1755 3827 50  0000 C CNN
+F 2 "" H 1750 4000 50  0001 C CNN
+F 3 "" H 1750 4000 50  0001 C CNN
+	1    1750 4000
+	1    0    0    -1
+$EndComp
+Wire Wire Line
+	1750 3950 1750 4000
 Wire Wire Line
 	5000 5700 5200 5700
@@
 Wire Wire Line
 	1650 5650 1650 5800
-NoConn ~ 1300 4450
 NoConn ~ 2500 4650
 Wire Wire Line
@@
 Text HLabel 1150 6350 0    50   Input ~ 0
 SDA
-Text Notes 950  5250 0    50   ~ 0
+Text Notes 1250 5300 0    50   ~ 0
 25MHz
 Wire Wire Line
@@
 Wire Wire Line
 	9100 4950 9100 5000
+Wire Wire Line
+	1600 4000 1250 4000
+Wire Wire Line
+	1250 4000 1250 4450
+Wire Wire Line
+	1250 4450 1300 4450
+Connection ~ 1600 4000
+Wire Wire Line
+	1600 4000 1600 3550
 $EndSCHEMATC
