File: connector.sch (KiCad schematic (older format))
At the start: 9 parts, among them J4 Conn_01x08, J5 Conn_01x06, J6 Conn_01x10, J7 Conn_01x08, U5 TA48L033

Commit message: BOM is ready
Parts:
- J4, J7: DigiKey (none) -> WM5543-ND
Changed lines of the file:
@@
 F 2 "Pin_Headers:Pin_Header_Straight_1x08_Pitch2.54mm" H 1950 1950 50  0001 C CNN
 F 3 "~" H 1950 1950 50  0001 C CNN
+F 4 "WM5543-ND" H 1950 1950 50  0001 C CNN "DigiKey"
 	1    1950 1950
 	-1   0    0    -1
@@
 F 2 "Pin_Headers:Pin_Header_Straight_1x08_Pitch2.54mm" H 7000 3450 50  0001 C CNN
 F 3 "~" H 7000 3450 50  0001 C CNN
+F 4 "WM5543-ND" H 7000 3450 50  0001 C CNN "DigiKey"
 	1    7000 3450
 	1    0    0    1
@@
 $EndComp
 $Comp
-L TA48L033:TA48L033 U5
-U 1 1 5F0FEF6E
-P 4050 2050
-F 0 "U5" H 4050 2292 50  0000 C CNN
-F 1 "TA48L033" H 4050 2201 50  0000 C CNN
-F 2 "TO_SOT_Packages_SMD:SOT-89-3_Handsoldering" H 4050 2250 50  0001 C CNN
-F 3 "https://toshiba.semicon-storage.com/jp/semiconductor/product/power-management-ics/detail.TA48L033F.html" H 4050 2000 50  0001 C CNN
-	1    4050 2050
-	1    0    0    -1
-$EndComp
-$Comp
-L Device:C C17
-U 1 1 5F0FF888
-P 3400 2300
-F 0 "C17" H 3515 2346 50  0000 L CNN
-F 1 "0.1u" H 3515 2255 50  0000 L CNN
-F 2 "Capacitors_THT:C_Disc_D4.7mm_W2.5mm_P5.00mm" H 3438 2150 50  0001 C CNN
-F 3 "~" H 3400 2300 50  0001 C CNN
-	1    3400 2300
-	1    0    0    -1
-$EndComp
-$Comp
-L Device:CP C16
-U 1 1 5F0FFE19
-P 3000 2300
-F 0 "C16" H 3118 2346 50  0000 L CNN
-F 1 "47u" H 3118 2255 50  0000 L CNN
-F 2 "Capacitors_THT:CP_Radial_D8.0mm_P2.50mm" H 3038 2150 50  0001 C CNN
-F 3 "~" H 3000 2300 50  0001 C CNN
-	1    3000 2300
-	1    0    0    -1
-$EndComp
-$Comp
-L Device:C C18
-U 1 1 5F100006
-P 4600 2300
-F 0 "C18" H 4715 2346 50  0000 L CNN
-F 1 "0.1u" H 4715 2255 50  0000 L CNN
-F 2 "Capacitors_THT:C_Disc_D4.7mm_W2.5mm_P5.00mm" H 4638 2150 50  0001 C CNN
-F 3 "~" H 4600 2300 50  0001 C CNN
-	1    4600 2300
-	1    0    0    -1
-$EndComp
-$Comp
-L Device:CP C19
-U 1 1 5F100230
-P 5000 2300
-F 0 "C19" H 5118 2346 50  0000 L CNN
-F 1 "47u" H 5118 2255 50  0000 L CNN
-F 2 "Capacitors_THT:CP_Radial_D8.0mm_P2.50mm" H 5038 2150 50  0001 C CNN
-F 3 "~" H 5000 2300 50  0001 C CNN
-	1    5000 2300
-	1    0    0    -1
-$EndComp
-$Comp
 L power:GND #PWR032
 U 1 1 5F104015
@@
 $EndComp
 $Comp
-L power:GND #PWR030
-U 1 1 5F1052CF
-P 3000 2650
-F 0 "#PWR030" H 3000 2400 50  0001 C CNN
-F 1 "GND" H 3005 2477 50  0000 C CNN
-F 2 "" H 3000 2650 50  0001 C CNN
-F 3 "" H 3000 2650 50  0001 C CNN
-	1    3000 2650
-	1    0    0    -1
-$EndComp
-$Comp
 L power:GND #PWR033
 U 1 1 5F1054A0
@@
 	1    0    0    -1
 $EndComp
-$Comp
-L power:GND #PWR034
-U 1 1 5F105733
-P 5000 2650
-F 0 "#PWR034" H 5000 2400 50  0001 C CNN
-F 1 "GND" H 5005 2477 50  0000 C CNN
-F 2 "" H 5000 2650 50  0001 C CNN
-F 3 "" H 5000 2650 50  0001 C CNN
-	1    5000 2650
-	1    0    0    -1
-$EndComp
-Wire Wire Line
-	5400 2050 5000 2050
 Wire Wire Line
 	3400 2150 3400 2050
 Connection ~ 3400 2050
 Wire Wire Line
-	3400 2050 3750 2050
-Wire Wire Line
-	3000 2150 3000 2050
-Connection ~ 3000 2050
-Wire Wire Line
-	3000 2050 3400 2050
-Wire Wire Line
 	4600 2050 4600 2150
 Connection ~ 4600 2050
@@
 	4600 2050 4350 2050
 Wire Wire Line
-	5000 2150 5000 2050
-Connection ~ 5000 2050
-Wire Wire Line
-	5000 2050 4600 2050
-Wire Wire Line
-	5000 2450 5000 2650
-Wire Wire Line
 	4600 2650 4600 2450
 Wire Wire Line
 	3400 2650 3400 2450
-Wire Wire Line
-	3000 2450 3000 2650
-Wire Wire Line
-	4050 2650 4050 2350
-Wire Wire Line
-	2150 2050 3000 2050
 Wire Wire Line
 	2150 2150 2650 2150
@@
 In the data sheet of TA48L033F, the pins are defined as :\n1. IN\n2. OUT\n3. GND\nTab. GND\n\nBut this definition doesn't fit to the SOT89-3 footprint \nof KiCAD. Thus, the pin assignment of the above symbol\nfollow the KiCAD SOT89-3.
 NoConn ~ 2150 1850
+Wire Wire Line
+	5000 2450 5000 2650
+Wire Wire Line
+	5000 2050 4600 2050
+Wire Wire Line
+	5400 2050 5000 2050
+Connection ~ 5000 2050
+Wire Wire Line
+	5000 2150 5000 2050
+$Comp
+L power:GND #PWR034
+U 1 1 5F105733
+P 5000 2650
+F 0 "#PWR034" H 5000 2400 50  0001 C CNN
+F 1 "GND" H 5005 2477 50  0000 C CNN
+F 2 "" H 5000 2650 50  0001 C CNN
+F 3 "" H 5000 2650 50  0001 C CNN
+	1    5000 2650
+	1    0    0    -1
+$EndComp
+Wire Wire Line
+	3000 2450 3000 2650
+$Comp
+L power:GND #PWR030
+U 1 1 5F1052CF
+P 3000 2650
+F 0 "#PWR030" H 3000 2400 50  0001 C CNN
+F 1 "GND" H 3005 2477 50  0000 C CNN
+F 2 "" H 3000 2650 50  0001 C CNN
+F 3 "" H 3000 2650 50  0001 C CNN
+	1    3000 2650
+	1    0    0    -1
+$EndComp
+Wire Wire Line
+	2150 2050 3000 2050
+Wire Wire Line
+	3000 2050 3400 2050
+Connection ~ 3000 2050
+Wire Wire Line
+	3000 2150 3000 2050
+Wire Wire Line
+	3400 2050 3750 2050
+Wire Wire Line
+	4050 2650 4050 2350
+$Comp
+L Device:C C18
+U 1 1 5F100006
+P 4600 2300
+F 0 "C18" H 4715 2346 50  0000 L CNN
+F 1 "0.1u" H 4715 2255 50  0000 L CNN
+F 2 "Capacitors_THT:C_Disc_D4.7mm_W2.5mm_P5.00mm" H 4638 2150 50  0001 C CNN
+F 3 "~" H 4600 2300 50  0001 C CNN
+	1    4600 2300
+	1    0    0    -1
+$EndComp
+$Comp
+L Device:CP C19
+U 1 1 5F100230
+P 5000 2300
+F 0 "C19" H 5118 2346 50  0000 L CNN
+F 1 "47u" H 5118 2255 50  0000 L CNN
+F 2 "Capacitors_THT:CP_Radial_D8.0mm_P2.50mm" H 5038 2150 50  0001 C CNN
+F 3 "~" H 5000 2300 50  0001 C CNN
+	1    5000 2300
+	1    0    0    -1
+$EndComp
+$Comp
+L Device:C C17
+U 1 1 5F0FF888
+P 3400 2300
+F 0 "C17" H 3515 2346 50  0000 L CNN
+F 1 "0.1u" H 3515 2255 50  0000 L CNN
+F 2 "Capacitors_THT:C_Disc_D4.7mm_W2.5mm_P5.00mm" H 3438 2150 50  0001 C CNN
+F 3 "~" H 3400 2300 50  0001 C CNN
+	1    3400 2300
+	1    0    0    -1
+$EndComp
+$Comp
+L Device:CP C16
+U 1 1 5F0FFE19
+P 3000 2300
+F 0 "C16" H 3118 2346 50  0000 L CNN
+F 1 "47u" H 3118 2255 50  0000 L CNN
+F 2 "Capacitors_THT:CP_Radial_D8.0mm_P2.50mm" H 3038 2150 50  0001 C CNN
+F 3 "~" H 3000 2300 50  0001 C CNN
+	1    3000 2300
+	1    0    0    -1
+$EndComp
+$Comp
+L TA48L033:TA48L033 U5
+U 1 1 5F0FEF6E
+P 4050 2050
+F 0 "U5" H 4050 2292 50  0000 C CNN
+F 1 "TA48L033" H 4050 2201 50  0000 C CNN
+F 2 "TO_SOT_Packages_SMD:SOT-89-3_Handsoldering" H 4050 2250 50  0001 C CNN
+F 3 "https://toshiba.semicon-storage.com/jp/semiconductor/product/power-management-ics/detail.TA48L033F.html" H 4050 2000 50  0001 C CNN
+	1    4050 2050
+	1    0    0    -1
+$EndComp
 $EndSCHEMATC

Commit message: update BOM
Parts:
- J4, J7: DigiKey WM5543-ND -> (none)
Changed lines of the file:
@@
 F 2 "Pin_Headers:Pin_Header_Straight_1x08_Pitch2.54mm" H 1950 1950 50  0001 C CNN
 F 3 "~" H 1950 1950 50  0001 C CNN
-F 4 "WM5543-ND" H 1950 1950 50  0001 C CNN "DigiKey"
+F 4 "" H 1950 1950 50  0001 C CNN "DigiKey"
 	1    1950 1950
 	-1   0    0    -1
@@
 F 2 "Pin_Headers:Pin_Header_Straight_1x08_Pitch2.54mm" H 7000 3450 50  0001 C CNN
 F 3 "~" H 7000 3450 50  0001 C CNN
-F 4 "WM5543-ND" H 7000 3450 50  0001 C CNN "DigiKey"
+F 4 "" H 7000 3450 50  0001 C CNN "DigiKey"
 	1    7000 3450
 	1    0    0    1

Commit message: Update readme
Parts:
- removed U5: TA48L033, TO_SOT_Packages_SMD:SOT-89-3_Handsoldering, symbol TA48L033:TA48L033
- added U5: TLV73333PDBV, TO_SOT_Packages_SMD:SOT-23-5_HandSoldering, symbol Regulator_Linear:TLV73333PDBV
Connections:
- wire segments 28 -> 32
Other:
- note removed: "In the data sheet of TA48L033F, the pins are defined as :\n1. IN\n2. OUT\n3. GND\nTab. GND\n\nBut this definition doesn't fit to the SOT89-3 footprint \nof KiCAD. Thus, the pin assignment of the above symbol\nfollow the KiCAD SOT89-3."
Changed lines of the file:
@@
 Text Notes 7300 3100 0    50   ~ 0
 J6 pin 5 is "rescue" pin for I2C SCL.\nIn case of some slave I2C SDA is stick to "L", \ntoggling SCL by this rescue pin can release the \nslave. \n\nThis rescue pin have to be configured as open \ndrain, and have to be kept as "H" during \nnormal operation. \n\nJ6 pin 5 is PA6 of Nucleo G431RB and F722ZE
-Text Notes 2650 3800 0    50   ~ 0
-In the data sheet of TA48L033F, the pins are defined as :\n1. IN\n2. OUT\n3. GND\nTab. GND\n\nBut this definition doesn't fit to the SOT89-3 footprint \nof KiCAD. Thus, the pin assignment of the above symbol\nfollow the KiCAD SOT89-3.
 NoConn ~ 2150 1850
 Wire Wire Line
@@
 	3000 2150 3000 2050
 Wire Wire Line
-	3400 2050 3750 2050
+	3400 2050 3650 2050
 Wire Wire Line
-	4050 2650 4050 2350
+	4050 2650 4050 2450
 $Comp
 L Device:C C18
@@
 $EndComp
 $Comp
-L TA48L033:TA48L033 U5
-U 1 1 5F0FEF6E
-P 4050 2050
-F 0 "U5" H 4050 2292 50  0000 C CNN
-F 1 "TA48L033" H 4050 2201 50  0000 C CNN
-F 2 "TO_SOT_Packages_SMD:SOT-89-3_Handsoldering" H 4050 2250 50  0001 C CNN
-F 3 "https://toshiba.semicon-storage.com/jp/semiconductor/product/power-management-ics/detail.TA48L033F.html" H 4050 2000 50  0001 C CNN
-	1    4050 2050
+L Regulator_Linear:TLV73333PDBV U5
+U 1 1 5F2FDED4
+P 4050 2150
+F 0 "U5" H 4050 2492 50  0000 C CNN
+F 1 "TLV73333PDBV" H 4050 2401 50  0000 C CNN
+F 2 "TO_SOT_Packages_SMD:SOT-23-5_HandSoldering" H 4050 2475 50  0001 C CIN
+F 3 "http://www.ti.com/lit/ds/symlink/tlv733p.pdf" H 4050 2150 50  0001 C CNN
+	1    4050 2150
 	1    0    0    -1
 $EndComp
+Wire Wire Line
+	3800 2150 3750 2150
+Wire Wire Line
+	3650 2150 3650 2050
+Connection ~ 3750 2150
+Wire Wire Line
+	3750 2150 3650 2150
+Connection ~ 3650 2050
+Wire Wire Line
+	3650 2050 3750 2050
 $EndSCHEMATC
